File: TVHR-PFG01.brd (EAGLE design)
At the start: 40.3 x 85.1 mm, 13 parts, among them IC1 NE556, X1 1502_01, X2 1502_01, X3 1502_01

Commit message: Many changes across the entire project
Parts:
- added IN: KLBR1, con-lumberg:KLBR1
- added POT3, POT4: 5K, pot:3RP/1610N
- renumbered R4 to POT1, R5 to POT2, X1 to OUT, X2 to CV2, X3 to CV1
Connections:
- new net N$13: CV2.2, POT4.1
- new net N$15: CV1.2, POT3.1
- new net N$24: IC1.8, IN.3
- net GND: now also IN.5, POT3.3, POT4.3
- net N$10: now also POT4.2; no longer CV2.2
- net N$6: now also IN.4; no longer IC1.8
- net N$9: now also POT3.2; no longer CV1.2
Changed lines of the file:
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@@
 <element name="C4" library="capacitor-wima" package="C2.5-3" value=".01uF" x="3.81" y="33.02"/>
 <element name="C5" library="capacitor-wima" package="C2.5-3" value=".01uF" x="20.32" y="33.02"/>
-<element name="R4" library="pot" package="3RP/1610N" value="500K" x="3.81" y="76.2" rot="R270.1"/>
-<element name="R5" library="pot" package="3RP/1610N" value="500K" x="36.83" y="76.2" rot="R90"/>
-<element name="X1" library="con-lumberg" package="1502_01" value="1502_01" x="20.32" y="6.35">
+<element name="POT1" library="pot" package="3RP/1610N" value="500K" x="3.81" y="76.2" rot="R270.1"/>
+<element name="POT2" library="pot" package="3RP/1610N" value="500K" x="36.83" y="76.2" rot="R90"/>
+<element name="OUT" library="con-lumberg" package="1502_01" value="1502_01" x="20.32" y="6.35">
 <attribute name="OC_NEWARK" value="unknown" x="60.96" y="-19.05" size="1.778" layer="27" display="off"/>
 <attribute name="MPN" value="" x="60.96" y="-19.05" size="1.778" layer="27" display="off"/>
@@
 <attribute name="OC_FARNELL" value="4739747" x="60.96" y="-19.05" size="1.778" layer="27" display="off"/>
 </element>
-<element name="X2" library="con-lumberg" package="1502_01" value="1502_01" x="34.29" y="6.35">
+<element name="CV2" library="con-lumberg" package="1502_01" value="1502_01" x="34.29" y="6.35">
 <attribute name="OC_NEWARK" value="unknown" x="53.34" y="-31.75" size="1.778" layer="27" display="off"/>
 <attribute name="MPN" value="" x="53.34" y="-31.75" size="1.778" layer="27" display="off"/>
@@
 <attribute name="OC_FARNELL" value="4739747" x="53.34" y="-31.75" size="1.778" layer="27" display="off"/>
 </element>
-<element name="X3" library="con-lumberg" package="1502_01" value="1502_01" x="6.35" y="6.35">
+<element name="CV1" library="con-lumberg" package="1502_01" value="1502_01" x="6.35" y="6.35">
 <attribute name="OC_NEWARK" value="unknown" x="38.1" y="-31.75" size="1.778" layer="27" display="off"/>
 <attribute name="MPN" value="" x="38.1" y="-31.75" size="1.778" layer="27" display="off"/>
@@
 <attribute name="OC_FARNELL" value="unknown" x="34.29" y="50.8" size="1.778" layer="27" rot="R90" display="off"/>
 </element>
+<element name="POT4" library="pot" package="3RP/1610N" value="5K" x="-19.05" y="13.97"/>
+<element name="POT3" library="pot" package="3RP/1610N" value="5K" x="-36.83" y="13.97"/>
+<element name="IN" library="con-lumberg" package="KLBR1" value="KLBR1" x="-53.34" y="-44.45">
+<attribute name="OC_NEWARK" value="97K2707" x="-53.34" y="-44.45" size="1.778" layer="27" display="off"/>
+<attribute name="MPN" value="KLBR 1" x="-53.34" y="-44.45" size="1.778" layer="27" display="off"/>
+<attribute name="MF" value="" x="-53.34" y="-44.45" size="1.778" layer="27" display="off"/>
+<attribute name="OC_FARNELL" value="1200140" x="-53.34" y="-44.45" size="1.778" layer="27" display="off"/>
+</element>
 </elements>
 <signals>
@@
 <contactref element="R1" pad="2"/>
 <contactref element="IC1" pad="1"/>
-<contactref element="R4" pad="3"/>
+<contactref element="POT1" pad="3"/>
 <wire x1="3.81" y1="71.12" x2="3.818725" y2="71.20000625" width="0.254" layer="16"/>
 <wire x1="8.89" y1="59.69" x2="16.51" y2="63.5" width="0" layer="19" extent="1-1"/>
@@
 <wire x1="2.54" y1="33.02" x2="8.89" y2="46.99" width="0" layer="19" extent="1-1"/>
 </signal>
-<signal name="N$6">
-<contactref element="IC1" pad="5"/>
-<contactref element="IC1" pad="8"/>
-<wire x1="8.89" y1="49.53" x2="16.51" y2="44.45" width="0" layer="19" extent="1-1"/>
-</signal>
 <signal name="N$4">
 <contactref element="IC1" pad="12"/>
 <contactref element="IC1" pad="13"/>
 <contactref element="C5" pad="1"/>
-<contactref element="R5" pad="1"/>
+<contactref element="POT2" pad="1"/>
 <wire x1="16.51" y1="57.15" x2="36.83" y2="71.2" width="0" layer="19" extent="1-1"/>
 <wire x1="16.51" y1="54.61" x2="16.51" y2="57.15" width="0" layer="19" extent="1-1"/>
@@
 <contactref element="R2" pad="2"/>
 <contactref element="R3" pad="2"/>
-<contactref element="X1" pad="2"/>
+<contactref element="OUT" pad="2"/>
 <wire x1="17.78" y1="26.67" x2="21.59" y2="26.67" width="0" layer="19" extent="1-1"/>
 <wire x1="17.97" y1="7.1" x2="17.78" y2="26.67" width="0" layer="19" extent="1-1"/>
@@
 <signal name="N$9">
 <contactref element="IC1" pad="3"/>
-<contactref element="X3" pad="2"/>
-<wire x1="4" y1="7.1" x2="8.89" y2="54.61" width="0" layer="19" extent="1-1"/>
+<contactref element="POT3" pad="2"/>
+<wire x1="-36.83" y1="13.97" x2="8.89" y2="54.61" width="0" layer="19" extent="1-1"/>
 </signal>
 <signal name="N$10">
 <contactref element="IC1" pad="11"/>
-<contactref element="X2" pad="2"/>
-<wire x1="31.94" y1="7.1" x2="16.51" y2="52.07" width="0" layer="19" extent="1-1"/>
+<contactref element="POT4" pad="2"/>
+<wire x1="-19.05" y1="13.97" x2="16.51" y2="52.07" width="0" layer="19" extent="1-1"/>
 </signal>
 <signal name="N$1">
@@
 <contactref element="SV1" pad="10"/>
 <contactref element="IC1" pad="7"/>
-<contactref element="X3" pad="1"/>
-<contactref element="X2" pad="1"/>
+<contactref element="CV2" pad="1"/>
 <contactref element="R3" pad="1"/>
-<contactref element="X1" pad="1"/>
+<contactref element="OUT" pad="1"/>
 <contactref element="C4" pad="2"/>
 <contactref element="C5" pad="2"/>
+<contactref element="POT4" pad="3"/>
+<contactref element="CV1" pad="1"/>
+<contactref element="POT3" pad="3"/>
+<contactref element="IN" pad="5"/>
 <wire x1="33.02" y1="57.15" x2="35.56" y2="57.15" width="0" layer="19" extent="1-1"/>
 <wire x1="35.56" y1="54.61" x2="35.56" y2="57.15" width="0" layer="19" extent="1-1"/>
@@
 <wire x1="5.08" y1="33.02" x2="21.59" y2="33.02" width="0" layer="19" extent="1-1"/>
 <wire x1="8.89" y1="44.45" x2="5.08" y2="33.02" width="0" layer="19" extent="1-1"/>
+<wire x1="-14.05" y1="13.97" x2="6.35" y2="8.7" width="0" layer="19" extent="1-1"/>
+<wire x1="-31.83" y1="13.97" x2="-14.05" y2="13.97" width="0" layer="19" extent="1-1"/>
+<wire x1="-53.34" y1="-39.75" x2="-31.83" y2="13.97" width="0" layer="19" extent="1-1"/>
 </signal>
 <signal name="+12V">
 <contactref element="IC1" pad="4"/>
-<contactref element="R4" pad="2"/>
-<contactref element="R5" pad="2"/>
+<contactref element="POT1" pad="2"/>
+<contactref element="POT2" pad="2"/>
 <contactref element="IC1" pad="10"/>
 <contactref element="IC1" pad="14"/>
@@
 <wire x1="3.81" y1="76.2" x2="16.51" y2="59.69" width="0" layer="19" extent="1-1"/>
 </signal>
+<signal name="N$13">
+<contactref element="CV2" pad="2"/>
+<contactref element="POT4" pad="1"/>
+<wire x1="-24.05" y1="13.97" x2="31.94" y2="7.1" width="0" layer="19" extent="1-1"/>
+</signal>
+<signal name="N$15">
+<contactref element="CV1" pad="2"/>
+<contactref element="POT3" pad="1"/>
+<wire x1="4" y1="7.1" x2="-41.83" y2="13.97" width="0" layer="19" extent="1-1"/>
+</signal>
+<signal name="N$24">
+<contactref element="IC1" pad="8"/>
+<contactref element="IN" pad="3"/>
+<wire x1="16.51" y1="44.45" x2="-53.34" y2="-49.15" width="0" layer="19" extent="1-1"/>
+</signal>
+<signal name="N$6">
+<contactref element="IN" pad="4"/>
+<contactref element="IC1" pad="5"/>
+<wire x1="8.89" y1="49.53" x2="-57.34" y2="-47.95" width="0" layer="19" extent="1-1"/>
+</signal>
 </signals>
