File: TVHR-PFG01.sch (EAGLE design)
At the start: 13 parts, among them IC1 NE556, X1 1502_01, X2 1502_01, X3 1502_01

Commit message: Many changes across the entire project
Parts:
- removed X2, X3: 1502_01, con-lumberg:1502_01
- added CV1, CV2: 1502_01, con-lumberg:1502_01
- added IN: KLBR1, con-lumberg:KLBR1
- added POT3, POT4: 5K, pot:3RP/1610N
- renumbered R4 to POT1, R5 to POT2, X1 to OUT
Connections:
- new net N$13: CV2.3, POT4.A
- new net N$15: CV1.3, POT3.A
- new net N$24: IC1.TRIG2, IN.3
- net GND: now also CV1.1, CV2.1, IN.5, POT3.E, POT4.E; no longer X2.1, X3.1
- net N$10: now also POT4.S; no longer X2.3
- net N$6: now also IN.4; no longer IC1.TRIG2
- net N$9: now also POT3.S; no longer X3.3
